File: sensorboard/sensorboard_copy.kicad_pcb (KiCad board)
At the start: 4 copper layers, 100 x 50 mm, 244 parts, among them J1 Conn_01x03, J10 Conn_01x02_Male, J11 Conn_01x05_Male, J12 Conn_01x03, J13 Conn_01x03, J14 USB_C_Receptacle_USB2.0, J2 Conn_01x03, J3 Conn_01x03, J4 Conn_01x03, J5 Conn_01x03, J6 Conn_01x03, J7 Conn_01x03, J8 Conn_01x03, J9 Conn_01x02_Male, Q1 MMDT2222A, U1 ESP32-PICO-D4, U10 MAX31856, U11 MAX31856, U12 RT9025-25GSP, U13 ADS1219, U14 ADS1219, U15 ADS1219, U16 MAX31856, U17 MAX31856, U18 MAX31856, U19 LTC4411, U2 LTC4411, U20 SN65HVD230, U3 TPS61092RSAR, U4 MAX31856, U5 MAX31856, U6 MAX31856, U7 MAX31856, U8 CP2102-GMR-QFN28, U9 MAX31856

Commit message: Update thermocouple connection
changed schematic (c55 --> cs5) and positions. Copies made
Parts:
- turned U1 to 90 degrees
Connections:
- TP1 pad 1: /CS3 -> /CS9
- TP10 pad 1: /CS7 -> /CS6
- TP11 pad 1: /CS5 -> /C55
- TP12 pad 1: /CS9 -> /CS4
- TP13 pad 1: /CS4 -> /CS3
- TP19 pad 1: /CS8 -> /CS2
- TP2 pad 1: /CS2 -> /CS8
- TP21 pad 1: /CS6 -> /CS0
- TP8 pad 1: /CS0 -> /BOOT
- TP9 pad 1: /BOOT -> /CS7
- U1 pad 14: /CS8 -> /CS2
- U1 pad 16: /CS6 -> /CS0
- U1 pad 17: /CS9 -> /CS4
- U1 pad 18: /CS7 -> /CS6
- U1 pad 20: /CS5 -> /C55
- U1 pad 21: /CS4 -> /CS3
- U1 pad 22: /CS3 -> /LED
- U1 pad 23: /CS0 -> /BOOT
- U1 pad 24: /CS2 -> unconnected-(U1-Pad24)
- U1 pad 28: unconnected-(U1-Pad28) -> /CS8
- U1 pad 29: /BOOT -> /CS7
- U1 pad 34: /LED -> /CS9
Routing:
- net /MOSI: track 129.4 -> 2.34 mm, vias 10 -> 1
- net /MISO: track 113.7 -> 2.37 mm, vias 10 -> 1
- net /SCLK: track 100.3 -> 2.07 mm, vias 10 -> 1
- net /CS7: track 38.5 -> 0.00 mm
- net /CS5: track 37.7 -> 0.00 mm
- net /CS9: track 31.1 -> 0.00 mm
- net /CS4: track 29.5 -> 0.00 mm
- net /CS6: track 23.5 -> 0.00 mm
- net /CS3: track 22.3 -> 0.00 mm
- net +3V3: track 67.9 -> 49.9 mm
- net /CS1: track 15.6 -> 0.00 mm
- net /CS0: track 14.4 -> 0.00 mm
- net /CS8: track 7.73 -> 0.00 mm
- net /CS2: track 7.36 -> 0.00 mm
