File: sensorboard/sensorboard_copy.kicad_sch (KiCad schematic)
At the start: 66 parts, among them J10 Conn_01x02_Male, J11 Conn_01x05_Male, J9 Conn_01x02_Male, Q1 MMDT2222A, U1 ESP32-PICO-D4, U2 LTC4411, U3 TPS61092RSAR

Commit message: Update thermocouple connection
changed schematic (c55 --> cs5) and positions. Copies made
Connections:
- net BOOT: now also TP8.1, U1.23 (IO0); no longer TP9.1, U1.29 (SD3/IO10)
- net CS0: now also TP21.1, U1.16 (IO27); no longer TP8.1, U1.23 (IO0)
- net CS2: now also TP19.1, U1.14 (IO25); no longer TP2.1, U1.24 (IO4)
- net CS3: now also TP13.1, U1.21 (IO15); no longer TP1.1, U1.22 (IO2)
- net CS4: now also TP12.1, U1.17 (IO14); no longer TP13.1, U1.21 (IO15)
- net CS5: no longer TP11.1, U1.20 (IO13)
- net CS6: now also TP10.1, U1.18 (IO12); no longer TP21.1, U1.16 (IO27)
- net CS7: now also TP9.1, U1.29 (SD3/IO10); no longer TP10.1, U1.18 (IO12)
- net CS8: now also TP2.1, U1.28 (SD2/IO9); no longer TP19.1, U1.14 (IO25)
- net CS9: now also TP1.1, U1.34 (IO5); no longer TP12.1, U1.17 (IO14)
- net LED: now also U1.22 (IO2); no longer U1.34 (IO5)
- new net C55: TP11.1, U1.20 (IO13)
- no-connect marks 37 -> 35
Other:
- moved on the sheet: TP1, TP2
