File: Sensors/Hardware/microSDcard.kicad_sch (KiCad schematic)
At the start: 2 parts, among them J16 Micro_SD_Card_Det

Commit message: rounding traces, ESD changes, boost footprints, removed drc exclusions
Parts:
- added C10: 0.1uF, Capacitor_SMD:C_0402_1005Metric, symbol Device:C_Small
Connections:
- net +3V3: now also C10.1
- net GND: now also C10.2
Changed lines of the file:
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@@
 (kicad_sch (version 20230121) (generator eeschema)
   (paper "A4")
+  (junction (at 138.43 81.28) (diameter 0) (color 0 0 0 0)
+  )
   (junction (at 143.51 116.84) (diameter 0) (color 0 0 0 0)
   )
@@
     (stroke (width 0) (type default))
   )
-  (wire (pts (xy 138.43 80.01) (xy 138.43 88.9))
+  (wire (pts (xy 138.43 80.01) (xy 138.43 81.28))
     (stroke (width 0) (type default))
   )
   (wire (pts (xy 153.67 91.44) (xy 154.94 91.44))
+    (stroke (width 0) (type default))
+  )
+  (wire (pts (xy 134.62 81.28) (xy 138.43 81.28))
     (stroke (width 0) (type default))
   )
@@
   )
   (wire (pts (xy 154.94 101.6) (xy 147.32 101.6))
+    (stroke (width 0) (type default))
+  )
+  (wire (pts (xy 138.43 81.28) (xy 138.43 88.9))
     (stroke (width 0) (type default))
   )
@@
     (effects (font (size 1.27 1.27)) (justify right))
   )
+  (symbol (lib_id "Device:C_Small") (at 134.62 83.82 0) (unit 1)
+    (in_bom yes) (on_board yes) (dnp no)
+    (property "Reference" "C10" (at 129.54 83.82 0)
+      (effects (font (size 1.27 1.27)))
+    )
+    (property "Value" "0.1uF" (at 129.54 86.1314 0)
+      (effects (font (size 1.27 1.27)))
+    )
+    (property "Footprint" "Capacitor_SMD:C_0402_1005Metric" (at 134.62 83.82 0)
+      (effects (font (size 1.27 1.27)) hide)
+    )
+    (property "Datasheet" "~" (at 134.62 83.82 0)
+      (effects (font (size 1.27 1.27)) hide)
+    )
+    (pin "1")
+    (pin "2")
+    (instances
+      (project "sensorboard"
+        (path "/26801cfb-b53b-4a6a-a2f4-5f4986565765"
+          (reference "C10") (unit 1)
+        )
+        (path "/26801cfb-b53b-4a6a-a2f4-5f4986565765/f50ea3f6-9887-4dc3-9ec9-7a0fb1ee7721"
+          (reference "C90") (unit 1)
+        )
+      )
+    )
+  )
+  (symbol (lib_id "power:GND") (at 134.62 86.36 0) (unit 1)
+    (in_bom yes) (on_board yes) (dnp no) (fields_autoplaced)
+    (property "Reference" "#PWR077" (at 134.62 92.71 0)
+      (effects (font (size 1.27 1.27)) hide)
+    )
+    (property "Value" "GND" (at 134.62 91.44 0)
+      (effects (font (size 1.27 1.27)))
+    )
+    (property "Footprint" "" (at 134.62 86.36 0)
+      (effects (font (size 1.27 1.27)) hide)
+    )
+    (property "Datasheet" "" (at 134.62 86.36 0)
+      (effects (font (size 1.27 1.27)) hide)
+    )
+    (pin "1")
+    (instances
+      (project "sensorboard"
+        (path "/26801cfb-b53b-4a6a-a2f4-5f4986565765/f50ea3f6-9887-4dc3-9ec9-7a0fb1ee7721"
+          (reference "#PWR077") (unit 1)
+        )
+      )
+    )
+  )
   (symbol (lib_id "Device:R_Small") (at 143.51 110.49 0) (unit 1)
