File: Hardware/Boosts.kicad_sch (KiCad schematic)
At the start: 43 parts, among them IC1 AP2205-W5-7, IC2 AP2205-W5-7, IC3 TPS61089RNRR, IC4 TPS61089RNRR

Commit message: Kermit Mini
Parts:
- removed C45 (x2): 10uF, Capacitor_SMD:C_0402_1005Metric, symbol Device:C_Small
- removed C49 (x2), C51, C87, C91, C92: 100nF, Capacitor_SMD:C_0402_1005Metric, symbol Device:C_Small
- removed C52: 47uF, Capacitor_SMD:C_1206_3216Metric, symbol Device:C_Small
- removed C53, C55: 10uF, Capacitor_SMD:C_0603_1608Metric, symbol Device:C_Small
- removed C54, C88, C89: 22uF, Capacitor_SMD:C_0805_2012Metric, symbol Device:C_Small
- removed C56: 120pF, Capacitor_SMD:C_0402_1005Metric, symbol Device:C_Small
- removed C57: 2.2nF, Capacitor_SMD:C_0805_2012Metric, symbol Device:C_Small
- removed C75, C80: 2.2uF, Capacitor_SMD:C_0402_1005Metric, symbol Device:C_Small
- removed C76, C78: 1uF, Capacitor_SMD:C_0402_1005Metric, symbol Device:C_Small
- removed C77: 180pF, Capacitor_SMD:C_0402_1005Metric, symbol Device:C_Small
- removed C79: 3.9nF, Capacitor_SMD:C_0402_1005Metric, symbol Device:C_Small
- removed C93: 22uF, Capacitor_SMD:C_1206_3216Metric, symbol Device:C_Small
- removed IC1, IC2: AP2205-W5-7, iclr:SOT95P282X145-5N, symbol iclr:AP2205-W5-7
- removed IC4: TPS61089RNRR, iclr:IC_TPS61089RNRR, symbol iclr:TPS61089RNRR
- removed L4, L5: SRR6038-5R0Y, iclr:SRR6038, symbol iclr:SRR6038-5R0Y
- removed R100: 475k, Resistor_SMD:R_0402_1005Metric, symbol Device:R_Small
- removed R101, R58: 360k, Resistor_SMD:R_0402_1005Metric, symbol Device:R_Small
- removed R102: 51k, Resistor_SMD:R_0402_1005Metric, symbol Device:R_Small
- removed R103: 287k, Resistor_SMD:R_0402_1005Metric, symbol Device:R_Small
- removed R21: 7.87k, Resistor_SMD:R_0402_1005Metric, symbol Device:R_Small
- removed R59: 100k, Resistor_SMD:R_0402_1005Metric, symbol Device:R_Small
- removed R62: 560k, Resistor_SMD:R_0402_1005Metric, symbol Device:R_Small
- removed R63: 309k, Resistor_SMD:R_0402_1005Metric, symbol Device:R_Small
- removed R64: 18.7k, Resistor_SMD:R_0402_1005Metric, symbol Device:R_Small
- removed R65: 953k, Resistor_SMD:R_0402_1005Metric, symbol Device:R_Small
- removed R97: 152k, Resistor_SMD:R_0603_1608Metric, symbol Device:R_Small
- removed R98: 50k, Resistor_SMD:R_0402_1005Metric, symbol Device:R_Small
- removed R99: 118k, Resistor_SMD:R_0402_1005Metric, symbol Device:R_Small
Connections:
- net at IC3.2 (VCC): no longer IC3.7 (EN)
- net +3V3: no longer names the net of IC3.9 (VIN)
- net FB_5V: no longer names the net of IC3.3 (FB)
- net GND: no longer names the net of IC3.5 (GND)
- net LDO5.5V_IN: no longer names the net of IC3.6 (VOUT)
- net SW_5V: no longer names the net of IC3.1 (FSW)
Other:
- note removed: "SIM: https://webench.ti.com/appinfo/webench/scripts/SDP.cgi?ID=0086ECB0F8B2BBA7"
- note removed: "SIM: https://webench.ti.com/appinfo/webench/scripts/SDP.cgi?ID=C25BB1AA15C31C1A"
- note removed: "Vout"

Commit message: wowwww
Parts:
- added C45 (x2): 10uF, Capacitor_SMD:C_0402_1005Metric, symbol Device:C_Small
- added C49 (x2), C51, C87, C91, C92: 100nF, Capacitor_SMD:C_0402_1005Metric, symbol Device:C_Small
- added C52: 47uF, Capacitor_SMD:C_1206_3216Metric, symbol Device:C_Small
- added C53, C55: 10uF, Capacitor_SMD:C_0603_1608Metric, symbol Device:C_Small
- added C54, C88, C89: 22uF, Capacitor_SMD:C_0805_2012Metric, symbol Device:C_Small
- added C56: 120pF, Capacitor_SMD:C_0402_1005Metric, symbol Device:C_Small
- added C57: 2.2nF, Capacitor_SMD:C_0805_2012Metric, symbol Device:C_Small
- added C75, C80: 2.2uF, Capacitor_SMD:C_0402_1005Metric, symbol Device:C_Small
- added C76, C78: 1uF, Capacitor_SMD:C_0402_1005Metric, symbol Device:C_Small
- added C77: 180pF, Capacitor_SMD:C_0402_1005Metric, symbol Device:C_Small
- added C79: 3.9nF, Capacitor_SMD:C_0402_1005Metric, symbol Device:C_Small
- added C93: 22uF, Capacitor_SMD:C_1206_3216Metric, symbol Device:C_Small
- added IC1, IC2: AP2205-W5-7, iclr:SOT95P282X145-5N, symbol iclr:AP2205-W5-7
- added IC4: TPS61089RNRR, iclr:IC_TPS61089RNRR, symbol iclr:TPS61089RNRR
- added L4, L5: SRR6038-5R0Y, iclr:SRR6038, symbol iclr:SRR6038-5R0Y
- added R100: 475k, Resistor_SMD:R_0402_1005Metric, symbol Device:R_Small
- added R101, R58: 360k, Resistor_SMD:R_0402_1005Metric, symbol Device:R_Small
- added R102: 51k, Resistor_SMD:R_0402_1005Metric, symbol Device:R_Small
- added R103: 287k, Resistor_SMD:R_0402_1005Metric, symbol Device:R_Small
- added R21: 7.87k, Resistor_SMD:R_0402_1005Metric, symbol Device:R_Small
- added R59: 100k, Resistor_SMD:R_0402_1005Metric, symbol Device:R_Small
- added R62: 560k, Resistor_SMD:R_0402_1005Metric, symbol Device:R_Small
- added R63: 309k, Resistor_SMD:R_0402_1005Metric, symbol Device:R_Small
- added R64: 18.7k, Resistor_SMD:R_0402_1005Metric, symbol Device:R_Small
- added R65: 953k, Resistor_SMD:R_0402_1005Metric, symbol Device:R_Small
- added R97: 152k, Resistor_SMD:R_0603_1608Metric, symbol Device:R_Small
- added R98: 50k, Resistor_SMD:R_0402_1005Metric, symbol Device:R_Small
- added R99: 118k, Resistor_SMD:R_0402_1005Metric, symbol Device:R_Small
Connections:
- net SW_5V: now reaches IC3.1 (FSW)
- net SW_5V: now also R63.1
- net at IC3.10 (BOOT): now also C87.1
- net at IC3.11 (SW): now also C87.2, L4.2, R63.2
- net at IC3.2 (VCC): now also IC3.7 (EN), C53.1
- net FB_5V: now reaches IC3.3 (FB)
- net FB_5V: now also R58.1, R59.2
- net at IC3.4 (COMP): now also C77.1, R21.1
- net GND: now reaches IC3.5 (GND)
- net GND: now also C45.2, C45.2, C49.2, C49.2, C51.2, C52.2, C53.2, C54.2, C55.2, C56.2, C57.2, C75.2, C76.2, C77.2, C78.2, C79.2, C80.2, C88.2, C89.2, C92.2, C93.2, IC1.2 (GND), IC2.2 (GND), IC4.5 (GND), R100.1, R102.1, R59.1, R62.1, R98.1, R99.1
- net LDO5.5V_IN: now reaches IC3.6 (VOUT)
- net LDO5.5V_IN: now also C45.1, C49.1, C54.1, C76.1, C88.1, IC1.1 (VIN), IC1.3 (EN), R58.2
- net at IC3.8 (ILIM): now also R62.2
- net +3V3: now reaches IC3.9 (VIN)
- net +3V3: now also C51.1, C52.1, C92.1, C93.1, IC4.9 (VIN), L4.1, L5.1
- new net: IC2.4 (ADJ/NC), R101.1, R102.2
- new net: C91.2, IC4.11 (SW), L5.2, R103.2
- new net: C57.1, R64.2
- new net: C55.1, IC4.2 (VCC), IC4.7 (EN)
- new net: C91.1, IC4.10 (BOOT)
- new net: C56.1, IC4.4 (COMP), R64.1
- new net: IC4.8 (ILIM), R100.2
- new net: IC1.4 (ADJ/NC), R97.1, R98.2
- new net: C79.1, R21.2
- new net 10V: C80.1, IC2.5 (VOUT), R101.2
- new net 5V: C75.1, IC1.5 (VOUT), R97.2
- new net FB_10V: IC4.3 (FB), R65.1, R99.2
- new net LDO11V_IN: C45.1, C49.1, C78.1, C89.1, IC2.1 (VIN), IC2.3 (EN), IC4.6 (VOUT), R65.2
- new net SW_10V: IC4.1 (FSW), R103.1
Other:
- note added: "Vout"
