File: Hardware/CAN_sch.kicad_sch (KiCad schematic)
At the start: 8 parts, among them U13 SN65HVD230

Commit message: wowwww
Connections:
- net Vref: now also JP37.1 (A)
Other:
- note added: "omitted Resistor"
Changed lines of the file:
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@@
+    (effects (font (size 1.27 1.27)) (justify left bottom))
+  )
+  (text "omitted Resistor \n" (at 76.2 97.79 0)
+    (effects (font (size 1.27 1.27)) (justify left bottom))
+  )
+  (label "Vref" (at 111.76 83.82 90) (fields_autoplaced)
     (effects (font (size 1.27 1.27)) (justify left bottom))
   )
