File: Hardware/NewMiniKermit.kicad_sch (KiCad schematic)
At the start: 24 parts, among them J3 Conn_01x06_Pin, U1 ESP32-S3, Y1 Crystal_GND24

Commit message: wowwww
Connections:
- net CAN+: now reaches J3.5 (Pin_5)
- net CAN-: now reaches J3.6 (Pin_6)
Other:
- removed sheet AnalogueSPI
- removed sheet Thermocouple1
- removed sheet Thermocouple2
- sheet Boosts ports: added 10V, 5V; removed none
- sheet CAN ports: added CAN_HIGH, CAN_LOW; removed none
