File: Hardware/power_sch.kicad_sch (KiCad schematic)
At the start: 14 parts, among them U6 LM66200DRLR, U7 MAX77827AEFD+T, U8 SC4215

Commit message: wowwww
Parts:
- added R17: 10k, Resistor_SMD:R_0402_1005Metric, symbol Device:R_Small
Connections:
- net at U6.8 (ST): now also R17.2
- new net VBUS: R17.1
Changed lines of the file:
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@@
+    (stroke (width 0) (type default))
+  )
+  (wire (pts (xy 72.39 63.5) (xy 73.66 63.5))
     (stroke (width 0) (type default))
   )
@@
     (stroke (width 0) (type default))
   )
+  (wire (pts (xy 67.31 58.42) (xy 67.31 63.5))
+    (stroke (width 0) (type default))
+  )
   (wire (pts (xy 106.68 63.5) (xy 110.49 63.5))
     (stroke (width 0) (type default))
   )
   (wire (pts (xy 101.6 63.5) (xy 106.68 63.5))
+    (stroke (width 0) (type default))
+  )
+  (wire (pts (xy 73.66 62.23) (xy 73.66 63.5))
     (stroke (width 0) (type default))
   )
@@
     )
   )
+  (symbol (lib_id "Device:R_Small") (at 69.85 63.5 270) (unit 1)
+    (in_bom yes) (on_board yes) (dnp no)
+    (property "Reference" "R17" (at 67.945 59.055 90)
+      (effects (font (size 1.27 1.27)) (justify left))
+    )
+    (property "Value" "10k" (at 67.945 61.5919 90)
+      (effects (font (size 1.27 1.27)) (justify left))
+    )
+    (property "Footprint" "Resistor_SMD:R_0402_1005Metric" (at 69.85 63.5 0)
+      (effects (font (size 1.27 1.27)) hide)
+    )
+    (property "Datasheet" "~" (at 69.85 63.5 0)
+      (effects (font (size 1.27 1.27)) hide)
+    )
+    (pin "1")
+    (pin "2")
+    (instances
+      (project "sensorboard"
+        (path "/26801cfb-b53b-4a6a-a2f4-5f4986565765/2b173291-6fb0-491b-9706-884a6390c6a8"
+          (reference "R17") (unit 1)
+        )
+      )
+      (project "NewMiniKermit"
+        (path "/b3ecbcce-8bc5-493c-b5b6-3e2f69f7358a/7aec0f76-f0ca-417c-88c2-9c2ae042aba1"
+          (reference "R15") (unit 1)
+        )
+      )
+    )
+  )
   (symbol (lib_id "power:GND") (at 71.12 50.8 180) (unit 1)
     (in_bom yes) (on_board yes) (dnp no) (fields_autoplaced)
@@
         )
       )
+    )
+  )
+  (symbol (lib_id "power:VBUS") (at 73.66 62.23 0) (unit 1)
+    (in_bom yes) (on_board yes) (dnp no) (fields_autoplaced)
+    (property "Reference" "#PWR062" (at 73.66 66.04 0)
+      (effects (font (size 1.27 1.27)) hide)
+    )
+    (property "Value" "VBUS" (at 73.66 57.15 0)
+      (effects (font (size 1.27 1.27)))
+    )
+    (property "Footprint" "" (at 73.66 62.23 0)
+      (effects (font (size 1.27 1.27)) hide)
+    )
+    (property "Datasheet" "" (at 73.66 62.23 0)
+      (effects (font (size 1.27 1.27)) hide)
+    )
+    (pin "1")
+    (instances
+      (project "NewMiniKermit"
+        (path "/b3ecbcce-8bc5-493c-b5b6-3e2f69f7358a/7aec0f76-f0ca-417c-88c2-9c2ae042aba1"
+          (reference "#PWR062") (unit 1)
+        )
+      )
