File: Hardware/analogueI2C.kicad_sch (KiCad schematic)
At the start: 138 parts, among them J10 1053131104, J11 1053131104, J12 1053131104, J13 1053131104, J14 1053131104, J3 1053131104, J4 1053131104, J5 1053131104, J6 1053131104, J7 1053131104, J8 1053131104, J9 1053131104, U10 ADS131M06IRSNR, U9 ADS131M06IRSNR

Commit message: Start work
Parts:
- removed C40: 1uF, Capacitor_SMD:C_0402_1005Metric, symbol Device:C_Small
- removed C42, C48: 0.1uF, Capacitor_SMD:C_0402_1005Metric, symbol Device:C_Small
- removed C44: 220nF, Capacitor_SMD:C_0402_1005Metric, symbol Device:C_Small
- removed C47: 10uF, Capacitor_SMD:C_0402_1005Metric, symbol Device:C_Small
- removed C50: 100nF, Capacitor_SMD:C_0402_1005Metric, symbol Device:C_Small
- removed C63, C64, C65, C66, C67, C68, C69, C70, C71, C72, C73, C74: 10nF, Capacitor_SMD:C_0402_1005Metric, symbol Device:C_Small
- removed J10, J11, J12, J13, J14, J3, J4, J5, J6, J7, J8, J9: 1053131104, iclr:1053131104, symbol iclr:1053131104
- removed JP1, JP11, JP12, JP13, JP14, JP15, JP16, JP18, JP2, JP22, JP23, JP24, JP25, JP26, JP27, JP28, JP3, JP33, JP34, JP35, JP36, JP38, JP39, JP4, JP7, JP9: SolderJumper_3_Open, Jumper:SolderJumper-3_P1.3mm_Open_RoundedPad1.0x1.5mm_NumberLabels, symbol Jumper:SolderJumper_3_Open
- removed JP10, JP17, JP19, JP20, JP21, JP29, JP30, JP31, JP32, JP5, JP6, JP8: SolderJumper_2_Open, Jumper:SolderJumper-2_P1.3mm_Open_RoundedPad1.0x1.5mm, symbol Jumper:SolderJumper_2_Open
- removed R22, R24, R26, R29, R34, R37, R39, R41, R48, R52: 6.2k, Resistor_SMD:R_0402_1005Metric, symbol Device:R_Small
- removed R23, R25, R27, R30, R35, R38, R40, R42, R49, R53: 12k, Resistor_SMD:R_0402_1005Metric, symbol Device:R_Small
- removed R28, R31, R32, R33, R36, R43, R44, R45, R55, R57: 32k, Resistor_SMD:R_0402_1005Metric, symbol Device:R_Small
- removed R46, R50: 6.04R, Resistor_SMD:R_0402_1005Metric, symbol Device:R_Small
- removed R47, R51, R54, R56: 15.8R, Resistor_SMD:R_0402_1005Metric, symbol Device:R_Small
- removed R60, R61: 49, Resistor_SMD:R_0402_1005Metric, symbol Device:R_Small
- removed R73, R74, R75, R76, R77, R78, R79, R80, R81, R82, R83, R84, R85, R86, R87, R88, R89, R90, R91, R92, R93, R94, R95, R96: 1k, Resistor_SMD:R_0402_1005Metric, symbol Device:R_Small
- removed U10: ADS131M06IRSNR, iclr:ADS131M06IRSNR, symbol iclr:ADS131M06IRSNR
Connections:
- no-connect marks 4 -> 2
Other:
- added sheet analog_in_3v3_0 (analog_input_3v3.kicad_sch)
- added sheet analog_in_3v3_1 (analog_input_3v3.kicad_sch)
- added sheet analog_in_5v10v_2 (analog_input_5v10v.kicad_sch)
- added sheet analog_in_5v10v_3 (analog_input_5v10v.kicad_sch)
- added sheet analog_in_5v10v_4 (analog_input_5v10v.kicad_sch)
- added sheet analog_in_5v10v_5 (analog_input_5v10v.kicad_sch)
- note removed: "10V option"
- note removed: "Added antialiasing filters for channel inputs"
- note removed: "Sensor inputs with 5V/3.3V input to 1.2V functionality"
- moved on the sheet: C39, C41, C43, C45, C46, C49, U9
