File: Hardware/power.kicad_sch (KiCad schematic)
At the start: 20 parts, among them U6 LM66200DRLR, U7 MAX77827AEFD+T, U8 SC4215

Commit message: Start of Kermit Mini
Parts:
- removed C31, C35, C37: 10uF, Capacitor_SMD:C_0402_1005Metric, symbol Device:C_Small
- removed C32: 10uF, Capacitor_SMD:C_0603_1608Metric, symbol Device:C_Small
- removed C33: 1uF, Capacitor_SMD:C_0402_1005Metric, symbol Device:C_Small
- removed C34: 22uF, Capacitor_SMD:C_0603_1608Metric, symbol Device:C_Small
- removed C36: 4.7uF, Capacitor_SMD:C_0402_1005Metric, symbol Device:C_Small
- removed C38: 0.1uF, Capacitor_SMD:C_0402_1005Metric, symbol Device:C_Small
- removed R18: 56k, Resistor_SMD:R_0402_1005Metric, symbol Device:R_Small
- removed R19: 10k, Resistor_SMD:R_0402_1005Metric, symbol Device:R_Small
- removed TP_3.3v1, TP_BBIN1, TP_BBOUT1, TP_RBUS1: TestPoint, TestPoint:TestPoint_Pad_D1.0mm, symbol Connector:TestPoint
- removed U6: LM66200DRLR, iclr:SOTFL50P160X60-8N, symbol iclr:LM66200DRLR
- removed U7: MAX77827AEFD+T, iclr:CONV_MAX77827AEFD+T, symbol iclr:MAX77827AEFD+T
- removed U8: SC4215, iclr:SOIC127P599X175-9N, symbol iclr:RT9025-25GSP
- added C20, C24, C26: 10uF, Capacitor_SMD:C_0402_1005Metric, symbol Device:C_Small
- added C21: 10uF, Capacitor_SMD:C_0603_1608Metric, symbol Device:C_Small
- added C22: 1uF, Capacitor_SMD:C_0402_1005Metric, symbol Device:C_Small
- added C23: 22uF, Capacitor_SMD:C_0603_1608Metric, symbol Device:C_Small
- added C25: 4.7uF, Capacitor_SMD:C_0402_1005Metric, symbol Device:C_Small
- added C27: 0.1uF, Capacitor_SMD:C_0402_1005Metric, symbol Device:C_Small
- added R14: 10k, Resistor_SMD:R_0402_1005Metric, symbol Device:R_Small
- added R15: 14k, Resistor_SMD:R_0402_1005Metric, symbol Device:R_Small
- added TP4, TP5, TP6, TP8: TestPoint, TestPoint:TestPoint_Pad_D1.5mm, symbol Connector:TestPoint
- added U3: LM66200DRLR, iclr:SOTFL50P160X60-8N, symbol iclr:LM66200DRLR
- added U4: MAX77827AEFD+T, iclr:CONV_MAX77827AEFD+T, symbol iclr:MAX77827AEFD+T
- added U5: SC4215, iclr:SOIC127P599X175-9N, symbol iclr:RT9025-25GSP
- R16: value 10k -> 56k
- R17: value 14k -> 10k
Connections:
- net +3V3: now also R16.1, C26.2, C27.2, TP6.1, U5.6 (VOUT)
- net BBIN: now also C20.1, C21.1, TP4.1, U3.2 (VOUT_1), U3.7 (VOUT_2), U4.3 (EN), U4.6 (IN)
- net BBOUT: now also C23.1, C24.1, C25.1, TP8.1, U4.11 (OUT), U4.13 (OUTS), U5.2 (EN), U5.3 (VIN)
- net BIAS: now also C22.1, U4.5 (BIAS)
- net FBIn: now also R16.2, R17.1, U5.7 (ADJ)
- net GND: now also C20.2, C21.2, C22.2, C23.2, C24.2, C25.2, C26.1, C27.1, R15.2, U3.1 (GND_1), U3.4 (~{ON}), U3.5 (GND_2), U4.4 (AGND), U4.9 (PGND), U5.8 (GND), U5.9 (GND)
- net LX1: now also U4.8 (LX1)
- net LX2: now also U4.10 (LX2)
- net RBUS_uC_V: now also TP5.1, U3.6 (VIN2)
- net SEL: now also R15.1, U4.1 (SEL); no longer R17.1
- net VBUS: now also R14.1, U3.3 (VIN1); no longer R16.1
- new net: R14.2, U3.8 (ST)

Commit message: Revert "Merge remote-tracking branch 'refs/remotes/origin/main'"
This reverts commit c9a99cb72454eddb78504ad976151236a8d13e5c, reversing
changes made to 3cdb2e540a9938f01cf78ecb1078cc5742e66bb5.
Parts:
- removed C20, C24, C26: 10uF, Capacitor_SMD:C_0402_1005Metric, symbol Device:C_Small
- removed C21: 10uF, Capacitor_SMD:C_0603_1608Metric, symbol Device:C_Small
- removed C22: 1uF, Capacitor_SMD:C_0402_1005Metric, symbol Device:C_Small
- removed C23: 22uF, Capacitor_SMD:C_0603_1608Metric, symbol Device:C_Small
- removed C25: 4.7uF, Capacitor_SMD:C_0402_1005Metric, symbol Device:C_Small
- removed C27: 0.1uF, Capacitor_SMD:C_0402_1005Metric, symbol Device:C_Small
- removed R14: 10k, Resistor_SMD:R_0402_1005Metric, symbol Device:R_Small
- removed R15: 14k, Resistor_SMD:R_0402_1005Metric, symbol Device:R_Small
- removed TP4, TP5, TP6, TP8: TestPoint, TestPoint:TestPoint_Pad_D1.5mm, symbol Connector:TestPoint
- removed U3: LM66200DRLR, iclr:SOTFL50P160X60-8N, symbol iclr:LM66200DRLR
- removed U4: MAX77827AEFD+T, iclr:CONV_MAX77827AEFD+T, symbol iclr:MAX77827AEFD+T
- removed U5: SC4215, iclr:SOIC127P599X175-9N, symbol iclr:RT9025-25GSP
- added C31, C35, C37: 10uF, Capacitor_SMD:C_0402_1005Metric, symbol Device:C_Small
- added C32: 10uF, Capacitor_SMD:C_0603_1608Metric, symbol Device:C_Small
- added C33: 1uF, Capacitor_SMD:C_0402_1005Metric, symbol Device:C_Small
- added C34: 22uF, Capacitor_SMD:C_0603_1608Metric, symbol Device:C_Small
- added C36: 4.7uF, Capacitor_SMD:C_0402_1005Metric, symbol Device:C_Small
- added C38: 0.1uF, Capacitor_SMD:C_0402_1005Metric, symbol Device:C_Small
- added R18: 56k, Resistor_SMD:R_0402_1005Metric, symbol Device:R_Small
- added R19: 10k, Resistor_SMD:R_0402_1005Metric, symbol Device:R_Small
- added TP_3.3v1, TP_BBIN1, TP_BBOUT1, TP_RBUS1: TestPoint, TestPoint:TestPoint_Pad_D1.0mm, symbol Connector:TestPoint
- added U6: LM66200DRLR, iclr:SOTFL50P160X60-8N, symbol iclr:LM66200DRLR
- added U7: MAX77827AEFD+T, iclr:CONV_MAX77827AEFD+T, symbol iclr:MAX77827AEFD+T
- added U8: SC4215, iclr:SOIC127P599X175-9N, symbol iclr:RT9025-25GSP
- R16: value 56k -> 10k
- R17: value 10k -> 14k
Connections:
- net +3V3: now also C37.2, C38.2, R18.1, TP_3.3v1.1, U8.6 (VOUT); no longer R16.1
- net BBIN: now also C31.1, C32.1, TP_BBIN1.1, U6.2 (VOUT_1), U6.7 (VOUT_2), U7.3 (EN), U7.6 (IN)
- net BBOUT: now also C34.1, C35.1, C36.1, TP_BBOUT1.1, U7.11 (OUT), U7.13 (OUTS), U8.2 (EN), U8.3 (VIN)
- net BIAS: now also C33.1, U7.5 (BIAS)
- net FBIn: now also R18.2, R19.1, U8.7 (ADJ); no longer R16.2, R17.1
- net GND: now also C31.2, C32.2, C33.2, C34.2, C35.2, C36.2, C37.1, C38.1, R19.2, U6.1 (GND_1), U6.4 (~{ON}), U6.5 (GND_2), U7.4 (AGND), U7.9 (PGND), U8.8 (GND), U8.9 (GND)
- net LX1: now also U7.8 (LX1)
- net LX2: now also U7.10 (LX2)
- net RBUS_uC_V: now also TP_RBUS1.1, U6.6 (VIN2)
- net SEL: now also R17.1, U7.1 (SEL)
- net VBUS: now also R16.1, U6.3 (VIN1)
- new net: R16.2, U6.8 (ST)
