File: Hardware/power.kicad_sch (KiCad schematic)
At the start: 20 parts, among them U3 LM66200DRLR, U4 MAX77827AEFD+T, U5 SC4215

Commit message: wrapping up layout
Parts:
- removed TP4, TP8: TestPoint, TestPoint:TestPoint_Pad_D1.5mm, symbol Connector:TestPoint
Changed lines of the file:
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@@
 	)
 	(junction
-		(at 123.19 52.07)
-		(diameter 0)
-		(color 0 0 0 0)
-	)
-	(junction
 		(at 240.03 60.96)
 		(diameter 0)
@@
 	(wire
 		(pts
-			(xy 123.19 52.07) (xy 128.27 52.07)
+			(xy 101.6 52.07) (xy 128.27 52.07)
 		)
 		(stroke
@@
 	(wire
 		(pts
-			(xy 101.6 52.07) (xy 123.19 52.07)
-		)
-		(stroke
-			(width 0)
-			(type default)
-		)
-	)
-	(wire
-		(pts
 			(xy 186.69 57.15) (xy 184.15 57.15)
 		)
@@
 		)
 		(instances
-			(project "RicardoTemplate"
+			(project "Ricardo-Kermit-Mini"
 				(path "/7db990e4-92e1-4f99-b4d2-435bbec1ba83/48a413b4-b7c2-44ac-971c-583c31b73475"
 					(reference "#PWR043")
@@
 		)
 		(instances
-			(project "RicardoTemplate"
+			(project "Ricardo-Kermit-Mini"
 				(path "/7db990e4-92e1-4f99-b4d2-435bbec1ba83/48a413b4-b7c2-44ac-971c-583c31b73475"
 					(reference "U3")
@@
 	)
 	(symbol
-		(lib_id "Connector:TestPoint")
-		(at 191.77 50.8 0)
-		(unit 1)
-		(exclude_from_sim no)
-		(in_bom yes)
-		(on_board yes)
-		(dnp no)
-		(property "Reference" "TP8"
-			(at 181.61 46.99 0)
-			(effects
-				(font
-					(size 1.27 1.27)
-				)
-				(justify left)
-			)
-		)
-		(property "Value" "TestPoint"
-			(at 181.61 49.5269 0)
-			(effects
-				(font
-					(size 1.27 1.27)
-				)
-				(justify left)
-			)
-		)
-		(property "Footprint" "TestPoint:TestPoint_Pad_D1.5mm"
-			(at 196.85 50.8 0)
-			(effects
-				(font
-					(size 1.27 1.27)
-				)
-				(hide yes)
-			)
-		)
-		(property "Datasheet" "~"
-			(at 196.85 50.8 0)
-			(effects
-				(font
-					(size 1.27 1.27)
-				)
-				(hide yes)
-			)
-		)
-		(property "Description" ""
-			(at 191.77 50.8 0)
-			(effects
-				(font
-					(size 1.27 1.27)
-				)
-				(hide yes)
-			)
-		)
-		(pin "1"
-		)
-		(instances
-			(project "RicardoTemplate"
-				(path "/7db990e4-92e1-4f99-b4d2-435bbec1ba83/48a413b4-b7c2-44ac-971c-583c31b73475"
-					(reference "TP8")
-					(unit 1)
-				)
-			)
-		)
-	)
-	(symbol
 		(lib_id "Device:R_Small")
 		(at 125.73 67.31 0)
@@
 		)
 		(instances
-			(project "RicardoTemplate"
+			(project "Ricardo-Kermit-Mini"
 				(path "/7db990e4-92e1-4f99-b4d2-435bbec1ba83/48a413b4-b7c2-44ac-971c-583c31b73475"
 					(reference "R15")
@@
 		)
 		(instances
-			(project "RicardoTemplate"
+			(project "Ricardo-Kermit-Mini"
 				(path "/7db990e4-92e1-4f99-b4d2-435bbec1ba83/48a413b4-b7c2-44ac-971c-583c31b73475"
 					(reference "C27")
@@
 		)
 		(instances
-			(project "RicardoTemplate"
+			(project "Ricardo-Kermit-Mini"
 				(path "/7db990e4-92e1-4f99-b4d2-435bbec1ba83/48a413b4-b7c2-44ac-971c-583c31b73475"
 					(reference "TP5")
@@
 		)
 		(instances
-			(project "RicardoTemplate"
+			(project "Ricardo-Kermit-Mini"
 				(path "/7db990e4-92e1-4f99-b4d2-435bbec1ba83/48a413b4-b7c2-44ac-971c-583c31b73475"
 					(reference "C24")
@@
 		)
 		(instances
-			(project "RicardoTemplate"
+			(project "Ricardo-Kermit-Mini"
 				(path "/7db990e4-92e1-4f99-b4d2-435bbec1ba83/48a413b4-b7c2-44ac-971c-583c31b73475"
 					(reference "#PWR036")
@@
 		)
 		(instances
-			(project "RicardoTemplate"
+			(project "Ricardo-Kermit-Mini"
 				(path "/7db990e4-92e1-4f99-b4d2-435bbec1ba83/48a413b4-b7c2-44ac-971c-583c31b73475"
 					(reference "L3")
@@
 		)
 		(instances
-			(project "RicardoTemplate"
+			(project "Ricardo-Kermit-Mini"
 				(path "/7db990e4-92e1-4f99-b4d2-435bbec1ba83/48a413b4-b7c2-44ac-971c-583c31b73475"
 					(reference "R14")
@@
 	)
 	(symbol
-		(lib_id "Connector:TestPoint")
-		(at 123.19 52.07 0)
-		(unit 1)
-		(exclude_from_sim no)
-		(in_bom yes)
-		(on_board yes)
-		(dnp no)
-		(property "Reference" "TP4"
-			(at 121.92 45.72 0)
-			(effects
-				(font
-					(size 1.27 1.27)
-				)
-				(justify left)
-			)
-		)
-		(property "Value" "TestPoint"
-			(at 121.92 43.1831 0)
-			(effects
-				(font
-					(size 1.27 1.27)
-				)
-				(justify left)
-			)
-		)
-		(property "Footprint" "TestPoint:TestPoint_Pad_D1.5mm"
-			(at 128.27 52.07 0)
-			(effects
-				(font
-					(size 1.27 1.27)
-				)
-				(hide yes)
-			)
-		)
-		(property "Datasheet" "~"
-			(at 128.27 52.07 0)
-			(effects
-				(font
-					(size 1.27 1.27)
-				)
-				(hide yes)
-			)
-		)
-		(property "Description" ""
-			(at 123.19 52.07 0)
-			(effects
-				(font
-					(size 1.27 1.27)
-				)
-				(hide yes)
-			)
-		)
-		(pin "1"
-		)
-		(instances
-			(project "RicardoTemplate"
-				(path "/7db990e4-92e1-4f99-b4d2-435bbec1ba83/48a413b4-b7c2-44ac-971c-583c31b73475"
-					(reference "TP4")
-					(unit 1)
-				)
-			)
-		)
-	)
-	(symbol
 		(lib_id "Device:R_Small")
 		(at 240.03 64.77 0)
@@
 		)
 		(instances
-			(project "RicardoTemplate"
+			(project "Ricardo-Kermit-Mini"
 				(path "/7db990e4-92e1-4f99-b4d2-435bbec1ba83/48a413b4-b7c2-44ac-971c-583c31b73475"
 					(reference "R17")
@@
 		)
 		(instances
-			(project "RicardoTemplate"
+			(project "Ricardo-Kermit-Mini"
 				(path "/7db990e4-92e1-4f99-b4d2-435bbec1ba83/48a413b4-b7c2-44ac-971c-583c31b73475"
 					(reference "#PWR045")
@@
 		)
 		(instances
-			(project "RicardoTemplate"
+			(project "Ricardo-Kermit-Mini"
 				(path "/7db990e4-92e1-4f99-b4d2-435bbec1ba83/48a413b4-b7c2-44ac-971c-583c31b73475"
 					(reference "C21")
@@
 		)
 		(instances
-			(project "RicardoTemplate"
+			(project "Ricardo-Kermit-Mini"
 				(path "/7db990e4-92e1-4f99-b4d2-435bbec1ba83/48a413b4-b7c2-44ac-971c-583c31b73475"
 					(reference "#PWR039")
@@
 		)
 		(instances
-			(project "RicardoTemplate"
+			(project "Ricardo-Kermit-Mini"
 				(path "/7db990e4-92e1-4f99-b4d2-435bbec1ba83/48a413b4-b7c2-44ac-971c-583c31b73475"
 					(reference "#PWR049")
@@
 		)
 		(instances
-			(project "RicardoTemplate"
+			(project "Ricardo-Kermit-Mini"
 				(path "/7db990e4-92e1-4f99-b4d2-435bbec1ba83/48a413b4-b7c2-44ac-971c-583c31b73475"
 					(reference "#PWR050")
@@
 		)
 		(instances
-			(project "RicardoTemplate"
+			(project "Ricardo-Kermit-Mini"
 				(path "/7db990e4-92e1-4f99-b4d2-435bbec1ba83/48a413b4-b7c2-44ac-971c-583c31b73475"
 					(reference "#PWR047")
@@
 		)
 		(instances
-			(project "RicardoTemplate"
+			(project "Ricardo-Kermit-Mini"
 				(path "/7db990e4-92e1-4f99-b4d2-435bbec1ba83/48a413b4-b7c2-44ac-971c-583c31b73475"
 					(reference "C26")
@@
 		)
 		(instances
-			(project "RicardoTemplate"
+			(project "Ricardo-Kermit-Mini"
 				(path "/7db990e4-92e1-4f99-b4d2-435bbec1ba83/48a413b4-b7c2-44ac-971c-583c31b73475"
 					(reference "#PWR041")
@@
 		)
 		(instances
-			(project "RicardoTemplate"
+			(project "Ricardo-Kermit-Mini"
 				(path "/7db990e4-92e1-4f99-b4d2-435bbec1ba83/48a413b4-b7c2-44ac-971c-583c31b73475"
 					(reference "TP6")
@@
 		)
 		(instances
-			(project "RicardoTemplate"
+			(project "Ricardo-Kermit-Mini"
 				(path "/7db990e4-92e1-4f99-b4d2-435bbec1ba83/48a413b4-b7c2-44ac-971c-583c31b73475"
 					(reference "U5")
@@
 		)
 		(instances
-			(project "RicardoTemplate"
+			(project "Ricardo-Kermit-Mini"
 				(path "/7db990e4-92e1-4f99-b4d2-435bbec1ba83/48a413b4-b7c2-44ac-971c-583c31b73475"
 					(reference "C20")
@@
 		)
 		(instances
-			(project "RicardoTemplate"
+			(project "Ricardo-Kermit-Mini"
 				(path "/7db990e4-92e1-4f99-b4d2-435bbec1ba83/48a413b4-b7c2-44ac-971c-583c31b73475"
 					(reference "U4")
@@
 		)
 		(instances
-			(project "RicardoTemplate"
+			(project "Ricardo-Kermit-Mini"
 				(path "/7db990e4-92e1-4f99-b4d2-435bbec1ba83/48a413b4-b7c2-44ac-971c-583c31b73475"
 					(reference "#PWR038")
@@
 		)
 		(instances
-			(project "RicardoTemplate"
+			(project "Ricardo-Kermit-Mini"
 				(path "/7db990e4-92e1-4f99-b4d2-435bbec1ba83/48a413b4-b7c2-44ac-971c-583c31b73475"
 					(reference "#PWR048")
@@
 		)
 		(instances
-			(project "RicardoTemplate"
+			(project "Ricardo-Kermit-Mini"
 				(path "/7db990e4-92e1-4f99-b4d2-435bbec1ba83/48a413b4-b7c2-44ac-971c-583c31b73475"
 					(reference "#PWR044")
@@
 		)
 		(instances
-			(project "RicardoTemplate"
+			(project "Ricardo-Kermit-Mini"
 				(path "/7db990e4-92e1-4f99-b4d2-435bbec1ba83/48a413b4-b7c2-44ac-971c-583c31b73475"
 					(reference "#PWR035")
@@
 		)
 		(instances
-			(project "RicardoTemplate"
+			(project "Ricardo-Kermit-Mini"
 				(path "/7db990e4-92e1-4f99-b4d2-435bbec1ba83/48a413b4-b7c2-44ac-971c-583c31b73475"
 					(reference "C25")
@@
 		)
 		(instances
-			(project "RicardoTemplate"
+			(project "Ricardo-Kermit-Mini"
 				(path "/7db990e4-92e1-4f99-b4d2-435bbec1ba83/48a413b4-b7c2-44ac-971c-583c31b73475"
 					(reference "C23")
@@
 		)
 		(instances
-			(project "RicardoTemplate"
+			(project "Ricardo-Kermit-Mini"
 				(path "/7db990e4-92e1-4f99-b4d2-435bbec1ba83/48a413b4-b7c2-44ac-971c-583c31b73475"
 					(reference "#PWR037")
@@
 		)
 		(instances
-			(project "RicardoTemplate"
+			(project "Ricardo-Kermit-Mini"
 				(path "/7db990e4-92e1-4f99-b4d2-435bbec1ba83/48a413b4-b7c2-44ac-971c-583c31b73475"
 					(reference "R16")
@@
 		)
 		(instances
-			(project "RicardoTemplate"
+			(project "Ricardo-Kermit-Mini"
 				(path "/7db990e4-92e1-4f99-b4d2-435bbec1ba83/48a413b4-b7c2-44ac-971c-583c31b73475"
 					(reference "#PWR040")
@@
 		)
 		(instances
-			(project "RicardoTemplate"
+			(project "Ricardo-Kermit-Mini"
 				(path "/7db990e4-92e1-4f99-b4d2-435bbec1ba83/48a413b4-b7c2-44ac-971c-583c31b73475"
 					(reference "C22")
@@
 		)
 		(instances
-			(project "RicardoTemplate"
+			(project "Ricardo-Kermit-Mini"
 				(path "/7db990e4-92e1-4f99-b4d2-435bbec1ba83/48a413b4-b7c2-44ac-971c-583c31b73475"
 					(reference "#PWR042")

Commit message: tidy up schematic and bom
Parts:
- C208: renamed from C27; value 0.1uF -> 100nF
- R201: renamed from R14; value 10k -> 10kΩ
- R202: renamed from R15; value 14k -> 14kΩ
- R203: renamed from R16; value 56k -> 56kΩ
- R204: renamed from R17; value 10k -> 10kΩ
- TP201: renamed from TP5; now left out of the parts list
- TP202: renamed from TP6; now left out of the parts list
- renumbered C20 to C201, C21 to C202, C22 to C203, C23 to C204, C24 to C205, C25 to C206, C26 to C207, L3 to L201, U3 to U201, U4 to U202, U5 to U203

Commit message: continued
Parts:
- U203: value SC4215 -> SC4215ASTRT
Changed lines of the file:
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@@
 		(fields_autoplaced yes)
 		(property "Reference" "U203"
-			(at 218.44 45.9572 0)
+			(at 218.44 44.45 0)
 			(effects
 				(font
@@
 			)
 		)
-		(property "Value" "SC4215"
-			(at 218.44 48.4941 0)
+		(property "Value" "SC4215ASTRT"
+			(at 218.44 46.99 0)
 			(effects
 				(font
