File: Hardware/sensorboard.kicad_sch (KiCad schematic)
At the start: 59 parts, among them J1 RBUS, U1 ESP32-S3, Y1 40MHz±10ppm

Commit message: Pinmap and ADC implementation update
need to sort out ledc
Other:
- note added: "TC0 in code"
- note added: "TC1 in code"
- note added: "TC2 in code"
- note added: "TC3 in code"
Changed lines of the file:
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@@
     (effects (font (size 2.54 2.54)) (justify right bottom))
+  )
+  (text "TC3 in code\n" (at 278.13 57.15 0)
+    (effects (font (size 1.27 1.27)) (justify left bottom))
   )
   (text "Dont use: integrated flash\n" (at 140.97 107.95 0)
@@
     (effects (font (size 1.27 1.27)) (justify left bottom))
   )
+  (text "TC2 in code" (at 276.86 40.64 0)
+    (effects (font (size 1.27 1.27)) (justify left bottom))
+  )
   (text "MainBoard\n" (at 187.96 190.5 0)
     (effects (font (size 1.27 1.27)) (justify left bottom))
@@
     (effects (font (size 1.27 1.27)) (justify left bottom))
   )
+  (text "TC1 in code" (at 275.59 24.13 0)
+    (effects (font (size 1.27 1.27)) (justify left bottom))
+  )
   (text "Controls JTAG source, don't use\n" (at 69.85 99.06 0)
     (effects (font (size 1.27 1.27)) (justify right bottom))
   )
   (text "Controls bootmode, don't use.\n" (at 140.97 135.89 0)
+    (effects (font (size 1.27 1.27)) (justify left bottom))
+  )
+  (text "TC0 in code" (at 275.59 73.66 0)
     (effects (font (size 1.27 1.27)) (justify left bottom))
   )
@@
   (symbol (lib_id "Connector:TestPoint") (at 72.39 147.32 90) (unit 1)
     (in_bom yes) (on_board yes) (dnp no)
-    (property "Reference" "TP_JTAG_MTMS1" (at 50.8 147.32 90)
+    (property "Reference" "TP_JTAG_MTMS1" (at 45.72 147.32 90)
       (effects (font (size 1.27 1.27)))
     )

Commit message: Start work
Other:
- note removed: "MainBoard"
- moved on the sheet: BOOTJUMPER1, C1, C10, C11, C12, C13, C14, C2, C3, C4, C5, C6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
