File: Hardware/thermocouple.kicad_sch (KiCad schematic)
At the start: 9 parts, among them U2 MAX31856

Commit message: Start work
Other:
- moved on the sheet: C15, C16, C17, C18, C61, R8, R9, TC2, U2
