File: Hardware/Ricardo-Kermit-Mini.kicad_sch (KiCad schematic)
At the start: 39 parts, among them J1 RBUS, J8 GPIO Breakout, U1 ESP32-S3, Y1 R940000171

Commit message: wrapping up layout
Parts:
- removed TP10, TP9, TP_CS1, TP_CS2: TestPoint, TestPoint:TestPoint_Pad_D1.0mm, symbol Connector:TestPoint
Connections:
- net +12V: no longer J1.4 (Pin_4), R7.1
- net ADS_CS0: now also U1.41 (GPIO36); no longer U1.42 (GPIO37)
- net CAN_RX: now also U1.47 (MTDI/JTAG/GPIO41)
- net CAN_TX: now also U1.48 (MTMS/JTAG/GPIO42)
- net CS0: now also U1.17 (GPIO12/ADC2_CH1); no longer U1.16 (GPIO11/ADC2_CH0)
- net CS1: now also U1.16 (GPIO11/ADC2_CH0); no longer U1.17 (GPIO12/ADC2_CH1)
- net GPIO8: now also J8.7 (Pin_7)
- net GPIO9: now also J8.8 (Pin_8)
- new net DEP: J1.4 (Pin_4), R7.1
- no-connect marks 8 -> 25

Commit message: layout
Parts:
- added CANRXLED1: CANRXLED, LED_SMD:LED_0402_1005Metric, symbol Device:LED_Small
- added CANTXLED1: CANTXLED, LED_SMD:LED_0402_1005Metric, symbol Device:LED_Small
- added R55, R56: 1k, Resistor_SMD:R_0402_1005Metric, symbol Device:R_Small
Connections:
- net 5V is gone; now on net +5V: J8.9 (Pin_9)
- net +3V3: now also R55.1, R56.1
- net CAN_RX: now also CANRXLED1.1 (K)
- net CAN_TX: now also CANTXLED1.1 (K)
- new net: CANTXLED1.2 (A), R55.2
- new net: CANRXLED1.2 (A), R56.2

Commit message: added diodes on gpio breakout and sensor supply
Parts:
- added D6: RCLAMP3346PQTNT, iclr:RCLAMP3346PQTNT, symbol iclr:RCLAMP3346PQTNT
- added TP3, TP4: TestPoint, TestPoint:TestPoint_Pad_D1.0mm, symbol Connector:TestPoint
Connections:
- net +3V3: now also J8.4 (Pin_4); no longer J8.5 (Pin_5)
- net +5V: now also J8.3 (Pin_3); no longer J8.9 (Pin_9)
- net CAN_RX: now also U1.44 (MTCK/JTAG/GPIO39); no longer U1.47 (MTDI/JTAG/GPIO41)
- net CAN_TX: now also U1.45 (MTDO/JTAG/GPIO40); no longer U1.48 (MTMS/JTAG/GPIO42)
- net GND: now also J8.2 (Pin_2), D6.2 (GND); no longer J8.10 (Pin_10)
- net GPIO4: now also J8.6 (Pin_6), D6.1 (K/A_1); no longer J8.2 (Pin_2)
- net GPIO5: now also J8.5 (Pin_5), D6.5 (K/A_4); no longer J8.3 (Pin_3)
- net GPIO6: now also J8.8 (Pin_8), D6.6 (K/A_5); no longer J8.4 (Pin_4)
- net GPIO7: now also J8.7 (Pin_7), D6.3 (K/A_2); no longer J8.6 (Pin_6)
- net GPIO8: now also J8.10 (Pin_10), D6.7 (K/A_6); no longer J8.7 (Pin_7)
- net GPIO9: now also J8.9 (Pin_9), D6.4 (K/A_3); no longer J8.8 (Pin_8)
- net RXD: now also TP4.1
- net TXD: now also TP3.1
Other:
- sheet Boosts1 renamed Boosts
- removed sheet thermocouple3
- added sheet thermocouple1 (thermocouple.kicad_sch)

Commit message: changes post 3rd review
Connections:
- net ADS_CS0: now also U1.42 (GPIO37); no longer U1.41 (GPIO36)
- new net ADS_DRDY: U1.41 (GPIO36)
- no-connect marks 25 -> 24
Other:
- sheet pressure_sensor1 ports: added ADS_DRDY; removed none
Changed lines of the file:
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@@
 	)
 	(no_connect
-		(at 135.89 105.41)
-	)
-	(no_connect
 		(at 207.01 139.7)
 	)
@@
 	(wire
 		(pts
+			(xy 214.63 87.884) (xy 223.52 87.884)
+		)
+		(stroke
+			(width 0)
+			(type default)
+		)
+	)
+	(wire
+		(pts
 			(xy 15.24 38.1) (xy 22.86 38.1)
 		)
@@
 	(wire
 		(pts
-			(xy 214.63 105.41) (xy 222.25 105.41)
+			(xy 214.63 108.458) (xy 222.25 108.458)
 		)
 		(stroke
@@
 	(wire
 		(pts
-			(xy 214.63 99.06) (xy 222.25 99.06)
+			(xy 214.63 102.108) (xy 222.25 102.108)
 		)
 		(stroke
@@
 	)
 	(label "ADS_CS0"
-		(at 135.89 102.87 0)
+		(at 135.89 105.41 0)
 		(fields_autoplaced yes)
 		(effects
@@
 		)
 	)
+	(label "ADS_DRDY"
+		(at 135.89 102.87 0)
+		(fields_autoplaced yes)
+		(effects
+			(font
+				(size 1.27 1.27)
+			)
+			(justify left bottom)
+		)
+	)
 	(label "CHIP_PU"
 		(at 36.83 165.1 180)
@@
 		)
 	)
+	(label "ADS_DRDY"
+		(at 223.52 87.884 0)
+		(fields_autoplaced yes)
+		(effects
+			(font
+				(size 1.27 1.27)
+			)
+			(justify left bottom)
+		)
+	)
 	(label "HSPI_MOSI"
 		(at 135.89 95.25 0)
@@
 	(symbol
 		(lib_id "power:+5V")
-		(at 222.25 105.41 0)
+		(at 222.25 108.458 0)
 		(unit 1)
 		(exclude_from_sim no)
@@
 		(fields_autoplaced yes)
 		(property "Reference" "#PWR016"
-			(at 222.25 109.22 0)
+			(at 222.25 112.268 0)
 			(effects
 				(font
@@
 		)
 		(property "Value" "+5V"
-			(at 222.25 100.33 0)
+			(at 222.25 103.378 0)
 			(effects
 				(font
@@
 		)
 		(property "Footprint" ""
-			(at 222.25 105.41 0)
+			(at 222.25 108.458 0)
 			(effects
 				(font
@@
 		)
 		(property "Datasheet" ""
-			(at 222.25 105.41 0)
+			(at 222.25 108.458 0)
 			(effects
 				(font
@@
 		)
 		(property "Description" ""
-			(at 222.25 105.41 0)
+			(at 222.25 108.458 0)
 			(effects
 				(font
@@
 		(lib_name "+12V_1")
 		(lib_id "power:+12V")
-		(at 222.25 99.06 0)
+		(at 222.25 102.108 0)
 		(unit 1)
 		(exclude_from_sim no)
@@
 		(fields_autoplaced yes)
 		(property "Reference" "#PWR09"
-			(at 222.25 102.87 0)
+			(at 222.25 105.918 0)
 			(effects
 				(font
@@
 		)
 		(property "Value" "+12V"
-			(at 222.25 93.98 0)
+			(at 222.25 97.028 0)
 			(effects
 				(font
@@
 		)
 		(property "Footprint" ""
-			(at 222.25 99.06 0)
+			(at 222.25 102.108 0)
 			(effects
 				(font
@@
 		)
 		(property "Datasheet" ""
-			(at 222.25 99.06 0)
+			(at 222.25 102.108 0)
 			(effects
 				(font
@@
 		)
 		(property "Description" ""
-			(at 222.25 99.06 0)
+			(at 222.25 102.108 0)
 			(effects
 				(font
@@
 	)
 	(sheet
-		(at 185.42 93.98)
+		(at 185.42 97.028)
 		(size 29.21 15.24)
 		(fields_autoplaced yes)
@@
 		)
 		(property "Sheetname" "Boosts"
-			(at 185.42 93.2684 0)
+			(at 185.42 96.3164 0)
 			(effects
 				(font
@@
 		)
 		(property "Sheetfile" "boosts_sch.kicad_sch"
-			(at 185.42 109.8046 0)
+			(at 185.42 112.8526 0)
 			(effects
 				(font
@@
 		)
 		(pin "12V" output
-			(at 214.63 99.06 0)
+			(at 214.63 102.108 0)
 			(effects
 				(font
@@
 		)
 		(pin "5V" output
-			(at 214.63 105.41 0)
+			(at 214.63 108.458 0)
 			(effects
 				(font
@@
 	(sheet
 		(at 185.42 72.39)
-		(size 29.21 13.97)
+		(size 29.21 17.526)
 		(fields_autoplaced yes)
 		(stroke
@@
 		)
 		(property "Sheetfile" "pressure_sensor_sch.kicad_sch"
-			(at 185.42 86.9446 0)
+			(at 185.42 90.5006 0)
 			(effects
 				(font
@@
 			(effects
 				(font
+					(size 1.27 1.27)
+				)
+				(justify right)
+			)
+		)
+		(pin "ADS_DRDY" output
+			(at 214.63 87.884 0)
+			(effects
+				(font

Commit message: post Andrei review, new SD
Connections:
- net ADS_CS0: now also U1.45 (MTDO/JTAG/GPIO40); no longer U1.42 (GPIO37)
- net ADS_DRDY: now also U1.44 (MTCK/JTAG/GPIO39); no longer U1.41 (GPIO36)
- net CAN_RX: now also U1.47 (MTDI/JTAG/GPIO41); no longer U1.44 (MTCK/JTAG/GPIO39)
- net CAN_TX: now also U1.48 (MTMS/JTAG/GPIO42); no longer U1.45 (MTDO/JTAG/GPIO40)
- net HSPI_MISO: now also U1.42 (GPIO37); no longer U1.39 (GPIO34)
- net HSPI_MOSI: now also U1.41 (GPIO36); no longer U1.38 (GPIO33)
- net HSPI_SCLK: now also U1.43 (GPIO38); no longer U1.40 (GPIO35)
- net SD1_CS: now also U1.36 (SPICLK_N/GPIO48); no longer U1.35 (SPID/GPIO32)
- net SD_EN: now also U1.27 (GPIO21); no longer U1.43 (GPIO38)
- net VSPI_MISO: now also U1.39 (GPIO34); no longer U1.32 (SPICS0/GPIO29)
- net VSPI_MOSI: now also U1.37 (SPICLK_P/GPIO47); no longer U1.34 (SPIQ/GPIO31)
- net VSPI_SCLK: now also U1.38 (GPIO33); no longer U1.33 (SPICLK/GPIO30)
- net at R54.2: now also U1.40 (GPIO35); no longer U1.37 (SPICLK_P/GPIO47)
- net SD_DET: now reaches U1.15 (GPIO10/ADC1_CH9)
- net SD1_DET: no longer names the net of U1.24 (GPIO18/ADC2_CH7/DAC_1)
Other:
- sheet microSD2 ports: added SD_DET; removed SD1_DET
- moved on the sheet: R54
Changed lines of the file:
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@@
 	)
 	(no_connect
+		(at 135.89 92.71)
+	)
+	(no_connect
 		(at 135.89 110.49)
 	)
 	(no_connect
+		(at 135.89 87.63)
+	)
+	(no_connect
 		(at 207.01 139.7)
 	)
 	(no_connect
-		(at 69.85 95.25)
+		(at 135.89 69.85)
 	)
 	(no_connect
-		(at 69.85 123.19)
+		(at 135.89 90.17)
 	)
 	(no_connect
@@
 	)
 	(no_connect
-		(at 69.85 125.73)
-	)
-	(no_connect
 		(at 69.85 74.93)
 	)
@@
 	)
 	(no_connect
-		(at 135.89 74.93)
-	)
-	(no_connect
 		(at 135.89 72.39)
 	)
@@
 	)
 	(no_connect
+		(at 135.89 85.09)
+	)
+	(no_connect
 		(at 135.89 77.47)
 	)
@@
 		(at 69.85 72.39)
 	)
-	(no_connect
-		(at 135.89 115.57)
-	)
 	(wire
 		(pts
@@
 	(wire
 		(pts
+			(xy 135.89 100.33) (xy 147.828 100.33)
+		)
+		(stroke
+			(width 0)
+			(type default)
+		)
+	)
+	(wire
+		(pts
 			(xy 160.02 127) (xy 156.21 127)
 		)
@@
 	(wire
 		(pts
-			(xy 189.992 55.88) (xy 193.04 55.88)
+			(xy 22.86 170.18) (xy 16.51 170.18)
 		)
 		(stroke
@@
 	(wire
 		(pts
-			(xy 22.86 170.18) (xy 16.51 170.18)
+			(xy 189.992 61.849) (xy 193.04 61.849)
 		)
 		(stroke
@@
 	(wire
 		(pts
-			(xy 189.992 61.849) (xy 193.04 61.849)
+			(xy 50.8 127) (xy 53.34 127)
 		)
 		(stroke
@@
 	(wire
 		(pts
-			(xy 50.8 127) (xy 53.34 127)
+			(xy 17.78 21.59) (xy 22.86 21.59)
 		)
 		(stroke
@@
 	(wire
 		(pts
-			(xy 17.78 21.59) (xy 22.86 21.59)
+			(xy 52.07 170.18) (xy 45.72 170.18)
 		)
 		(stroke
@@
 	(wire
 		(pts
-			(xy 52.07 170.18) (xy 45.72 170.18)
+			(xy 214.63 74.93) (xy 223.52 74.93)
 		)
 		(stroke
@@
 	(wire
 		(pts
-			(xy 214.63 74.93) (xy 223.52 74.93)
+			(xy 66.04 100.33) (xy 69.85 100.33)
 		)
 		(stroke
@@
 	(wire
 		(pts
-			(xy 66.04 100.33) (xy 69.85 100.33)
+			(xy 189.992 55.372) (xy 193.04 55.372)
 		)
 		(stroke
@@
 	)
 	(label "ADS_CS0"
-		(at 135.89 105.41 0)
+		(at 69.85 120.65 180)
 		(fields_autoplaced yes)
 		(effects
@@
 				(size 1.27 1.27)
 			)
-			(justify left bottom)
+			(justify right bottom)
 		)
 	)
@@
 	)
 	(label "VSPI_MISO"
-		(at 135.89 85.09 0)
+		(at 135.89 97.79 0)
 		(fields_autoplaced yes)
 		(effects
@@
 	)
 	(label "ADS_DRDY"
-		(at 135.89 102.87 0)
+		(at 69.85 118.11 180)
 		(fields_autoplaced yes)
 		(effects
@@
 				(size 1.27 1.27)
 			)
-			(justify left bottom)
+			(justify right bottom)
+		)
+	)
+	(label "SD_DET"
+		(at 69.85 95.25 180)
+		(fields_autoplaced yes)
+		(effects
+			(font
+				(size 1.27 1.27)
+			)
+			(justify right bottom)
 		)
 	)
@@
 	)
 	(label "ADS_CLK"
-		(at 140.97 118.11 0)
+		(at 152.908 100.33 0)
 		(fields_autoplaced yes)
 		(effects
@@
 	)
 	(label "HSPI_MOSI"
-		(at 135.89 95.25 0)
+		(at 135.89 102.87 0)
 		(fields_autoplaced yes)
 		(effects
@@
 	)
 	(label "HSPI_SCLK"
-		(at 135.89 100.33 0)
+		(at 135.89 107.95 0)
 		(fields_autoplaced yes)
 		(effects
@@
 	)
 	(label "SD_EN"
-		(at 135.89 107.95 0)
+		(at 135.89 74.93 0)
 		(fields_autoplaced yes)
 		(effects
@@
 	)
 	(label "SD1_CS"
-		(at 135.89 92.71 0)
+		(at 135.89 115.57 0)
 		(fields_autoplaced yes)
 		(effects
@@
 	)
 	(label "VSPI_SCLK"
-		(at 135.89 87.63 0)
+		(at 135.89 95.25 0)
 		(fields_autoplaced yes)
 		(effects
@@
 	)
 	(label "CAN_RX"
-		(at 69.85 118.11 180)
+		(at 69.85 123.19 180)
 		(fields_autoplaced yes)
 		(effects
@@
 	)
 	(label "HSPI_MISO"
-		(at 135.89 97.79 0)
+		(at 135.89 105.41 0)
 		(fields_autoplaced yes)
 		(effects
@@
 		)
 	)
-	(label "GPIO7"
-		(at 191.008 28.702 180)
+	(label "SD_DET"
+		(at 189.992 55.372 180)
 		(fields_autoplaced yes)
 		(effects
@@
 		)
 	)
-	(label "HSPI_SCLK"
-		(at 179.07 120.65 0)
-		(fields_autoplaced yes)
-		(effects
-			(font
-				(size 1.27 1.27)
-			)
-			(justify left bottom)
-		)
-	)
-	(label "SD1_DET"
-		(at 189.992 55.88 180)
+	(label "GPIO7"
+		(at 191.008 28.702 180)
 		(fields_autoplaced yes)
 		(effects
@@
 		)
 	)
-	(label "SD1_DET"
-		(at 135.89 69.85 0)
+	(label "HSPI_SCLK"
+		(at 179.07 120.65 0)
 		(fields_autoplaced yes)
 		(effects
@@
 	)
 	(label "VSPI_MOSI"
-		(at 135.89 90.17 0)
+		(at 135.89 118.11 0)
 		(fields_autoplaced yes)
 		(effects
@@
 	)
 	(label "CAN_TX"
-		(at 69.85 120.65 180)
+		(at 69.85 125.73 180)
 		(fields_autoplaced yes)
 		(effects
@@
 	(symbol
 		(lib_id "Device:R_Small")
-		(at 138.43 118.11 270)
+		(at 150.368 100.33 270)
 		(mirror x)
 		(unit 1)
@@
 		(dnp no)
 		(property "Reference" "R54"
-			(at 138.43 116.078 90)
+			(at 150.368 98.298 90)
 			(effects
 				(font
@@
 		)
 		(property "Value" "54.9R"
-			(at 138.684 120.142 90)
+			(at 150.622 102.362 90)
 			(effects
 				(font
@@
 		)
 		(property "Footprint" "Resistor_SMD:R_0402_1005Metric"
-			(at 138.43 118.11 0)
+			(at 150.368 100.33 0)
 			(effects
 				(font
@@
 		)
 		(property "Datasheet" "~"
-			(at 138.43 118.11 0)
+			(at 150.368 100.33 0)
 			(effects
 				(font
@@
 		)
 		(property "Description" ""
-			(at 138.43 118.11 0)
+			(at 150.368 100.33 0)
 			(effects
 				(font
@@
 			)
 		)
-		(pin "SD1_DET" input
-			(at 193.04 55.88 180)
-			(effects
-				(font
-					(size 1.27 1.27)
-				)
-				(justify left)
-			)
-		)
 		(pin "VSPI_SCLK" input
 			(at 193.04 52.07 180)
@@
 			(effects
 				(font
+					(size 1.27 1.27)
+				)
+				(justify left)
+			)
+		)
+		(pin "SD_DET" input
+			(at 193.04 55.372 180)
+			(effects
+				(font

Commit message: Ordering
Parts:
- R6: MPN (none) -> AC0402FR-07499RL
Changed lines of the file:
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@@
+			)
+		)
+		(property "MPN" "AC0402FR-07499RL"
+			(at 67.31 113.03 90)
+			(effects
+				(font
+					(size 1.27 1.27)
+				)
+				(hide yes)
 			)
 		)

Commit message: currently in the basket
Parts:
- CANRXLED1: value CANRXLED -> AMBER_LED
- CANTXLED1: value CANTXLED -> EMERALD_LED
Changed lines of the file:
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@@
 			)
 		)
-		(property "Value" "CANTXLED"
+		(property "Value" "EMERALD_LED"
 			(at 25.4 40.9956 0)
 			(effects
@@
 			)
 		)
-		(property "Value" "CANRXLED"
+		(property "Value" "AMBER_LED"
 			(at 25.4 53.6956 0)
 			(effects
