File: Hardware/Ricardo-Kermit-Mini.kicad_sch (KiCad schematic)
At the start: 42 parts, among them J1 RBUS, J8 GPIO Breakout, U1 ESP32-S3, Y1 R940000171

Commit message: tidy up schematic and bom
Parts:
- C103: renamed from C3; value 0.1uF -> 100nF
- C105: renamed from C5; value 0.1uF -> 100nF
- C106: renamed from C6; value 0.1uF -> 100nF
- C108: renamed from C8; value 0.1uF -> 100nF
- C110: renamed from C10; value 0.1uF -> 100nF
- C111: renamed from C11; value 0.1uF -> 100nF
- D101: renamed from TXLED1; value GREEN_LED -> LED_GREEN
- D102: renamed from CANTXLED1; value EMERALD_LED -> LED_GREEN
- D103: renamed from CANRXLED1; value AMBER_LED -> LED_ORANGE
- D104: renamed from 3V3LED1; value BLUE_LED -> LED_BLUE
- D105: renamed from 12VLED1; value RED_LED -> LED_RED
- H101: renamed from H1; now left out of the parts list
- H102: renamed from H2; now left out of the parts list
- H103: renamed from H3; now left out of the parts list
- H104: renamed from H4; now left out of the parts list
- L101: renamed from L1; value 2.0nH -> 2nH
- R101: renamed from R1; value 10K -> 10kΩ
- R102: renamed from R2; value 470 -> 470Ω
- R103: renamed from R55; value 1k -> 1kΩ
- R104: renamed from R56; value 1k -> 1kΩ
- R105: renamed from R3; value 10K -> 10kΩ
- R106: renamed from R4; value 470 -> 470Ω
- R107: renamed from R6; value 499R -> 499Ω
- R108: renamed from R7; value 3k -> 3kΩ
- R109: renamed from R54; value 54.9R -> 54.9Ω
- TP101: renamed from TP4; now left out of the parts list
- TP102: renamed from TP3; now left out of the parts list
- Y101: renamed from Y1; value R940000171 -> 40MHz; MPN (none) -> R940000171
- renumbered C1 to C101, C2 to C102, C4 to C104, C7 to C107, C9 to C109, C13 to C112, C14 to C113, D6 to D106, ENJUMPER1 to J101, BOOTJUMPER1 to J102, J1 to J103, J8 to J104, L2 to L102, U1 to U101

Commit message: continued
Parts:
- D101, D104, D105: footprint Resistor_SMD:R_0402_1005Metric -> LED_SMD:LED_0402_1005Metric
- Y101: value 40MHz -> 40MHz±10ppm
Changed lines of the file:
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@@
 			)
 		)
-		(property "Footprint" "Resistor_SMD:R_0402_1005Metric"
+		(property "Footprint" "LED_SMD:LED_0402_1005Metric"
 			(at 25.4 21.59 90)
 			(effects
@@
 			)
 		)
-		(property "Footprint" "Resistor_SMD:R_0402_1005Metric"
+		(property "Footprint" "LED_SMD:LED_0402_1005Metric"
 			(at 54.61 21.59 90)
 			(effects
@@
 			)
 		)
-		(property "Footprint" "Resistor_SMD:R_0402_1005Metric"
+		(property "Footprint" "LED_SMD:LED_0402_1005Metric"
 			(at 63.5 26.67 90)
 			(effects
@@
 			)
 		)
-		(property "Value" "40MHz"
+		(property "Value" "40MHz±10ppm"
 			(at 152.4 124.46 90)
 			(effects
