File: Hardware/pressure_sensor_sch.kicad_sch (KiCad schematic)
At the start: 56 parts, among them IC5 ADS131M04IRUKR, J4 1053131104, J5 1053131104, J6 1053131104, J7 1053131104

Commit message: tidy up schematic and bom
Parts:
- JP701: renamed from JP3; now left out of the parts list
- JP702: renamed from JP6; now left out of the parts list
- JP703: renamed from JP4; now left out of the parts list
- JP704: renamed from JP7; now left out of the parts list
- JP705: renamed from JP5; now left out of the parts list
- JP706: renamed from JP19; now left out of the parts list
- JP708: renamed from JP13; now left out of the parts list
- JP710: renamed from JP10; now left out of the parts list
- JP711: renamed from JP11; now left out of the parts list
- JP712: renamed from JP14; now left out of the parts list
- JP713: renamed from JP12; now left out of the parts list
- JP714: renamed from JP17; now left out of the parts list
- JP715: renamed from JP15; now left out of the parts list
- JP716: renamed from JP18; now left out of the parts list
- JP719: renamed from JP20; now left out of the parts list
- JP720: renamed from JP22; now left out of the parts list
- R701: renamed from R34; value 75k -> 75kΩ
- R702: renamed from R36; value 14k -> 14kΩ
- R703: renamed from R38; value 10k -> 10kΩ
- R704: renamed from R35; value 75k -> 75kΩ
- R705: renamed from R39; value 14k -> 14kΩ
- R706: renamed from R37; value 10k -> 10kΩ
- R707: renamed from R40; value 1k -> 1kΩ
- R708: renamed from R57; value 1k -> 1kΩ
- R709: renamed from R44; value 49.9 -> 49.9Ω
- R710: renamed from R45; value 1k -> 1kΩ
- R711: renamed from R41; value 49.9 -> 49.9Ω
- R712: renamed from R58; value 1k -> 1kΩ
- R713: renamed from R42; value 75k -> 75kΩ
- R714: renamed from R43; value 14k -> 14kΩ
- R715: renamed from R46; value 10k -> 10kΩ
- R716: renamed from R47; value 75k -> 75kΩ
- R717: renamed from R49; value 14k -> 14kΩ
- R718: renamed from R61; value 10k -> 10kΩ
- R719: renamed from R48; value 1k -> 1kΩ
- R720: renamed from R62; value 1k -> 1kΩ
- R721: renamed from R59; value 49.9 -> 49.9Ω
- R722: renamed from R63; value 49.9 -> 49.9Ω
- R723: renamed from R60; value 1k -> 1kΩ
- R724: renamed from R64; value 1k -> 1kΩ
- renumbered C50 to C701, C51 to C702, C52 to C703, C65 to C704, C63 to C705, C64 to C706, C66 to C707, J4 to J701, J5 to J702, J6 to J703, J7 to J704, JP9 to JP707, JP8 to JP709, JP16 to JP717, JP23 to JP718, IC5 to U701
