File: Hardware/usb.kicad_sch (KiCad schematic)
At the start: 8 parts, among them J2 USB_C_Receptacle_USB2.0

Commit message: layout
Changed lines of the file:
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@@
+	(wire
+		(pts
+			(xy 150.876 91.44) (xy 150.876 92.71)
+		)
+		(stroke
+			(width 0)
+			(type default)
+		)
+	)
 	(wire
 		(pts
@@
 	(wire
 		(pts
+			(xy 152.4 92.71) (xy 150.876 92.71)
+		)
+		(stroke
+			(width 0)
+			(type default)
+		)
+	)
+	(wire
+		(pts
 			(xy 125.73 99.06) (xy 125.73 96.52)
 		)
@@
 	(wire
 		(pts
-			(xy 125.73 96.52) (xy 127 96.52)
+			(xy 125.73 96.52) (xy 128.778 96.52)
 		)
 		(stroke
@@
 		(pts
 			(xy 118.11 99.06) (xy 120.65 99.06)
+		)
+		(stroke
+			(width 0)
+			(type default)
+		)
+	)
+	(wire
+		(pts
+			(xy 128.778 96.52) (xy 128.778 96.774)
 		)
 		(stroke
@@
 	(symbol
 		(lib_id "power:GND")
-		(at 127 96.52 90)
+		(at 128.778 96.774 0)
 		(unit 1)
 		(exclude_from_sim no)
@@
 		(dnp no)
 		(property "Reference" "#PWR031"
-			(at 133.35 96.52 0)
+			(at 128.778 103.124 0)
 			(effects
 				(font
@@
 		)
 		(property "Value" "GND"
-			(at 130.2512 96.393 90)
+			(at 128.905 100.0252 90)
 			(effects
 				(font
@@
 		)
 		(property "Footprint" ""
-			(at 127 96.52 0)
+			(at 128.778 96.774 0)
 			(effects
 				(font
@@
 		)
 		(property "Datasheet" ""
-			(at 127 96.52 0)
-			(effects
-				(font
-					(size 1.27 1.27)
-				)
-				(hide yes)
-			)
-		)
-		(property "Description" ""
-			(at 127 96.52 0)
+			(at 128.778 96.774 0)
+			(effects
+				(font
+					(size 1.27 1.27)
+				)
+				(hide yes)
+			)
+		)
+		(property "Description" ""
+			(at 128.778 96.774 0)
 			(effects
 				(font
@@
 		(dnp no)
 		(property "Reference" "R12"
-			(at 129.54 100.33 90)
+			(at 124.968 101.092 90)
 			(effects
 				(font
@@
 		)
 		(property "Value" "5.1k"
-			(at 129.54 102.6414 90)
+			(at 124.968 103.4034 90)
 			(effects
 				(font
@@
 	(symbol
 		(lib_id "power:GND")
-		(at 165.1 92.71 90)
+		(at 165.1 92.71 0)
 		(unit 1)
 		(exclude_from_sim no)
@@
 		(dnp no)
 		(property "Reference" "#PWR034"
-			(at 171.45 92.71 0)
+			(at 165.1 99.06 0)
 			(effects
 				(font
@@
 		)
 		(property "Value" "GND"
-			(at 168.3512 92.583 90)
+			(at 165.227 95.9612 90)
 			(effects
 				(font
@@
 	(symbol
 		(lib_id "power:VBUS")
-		(at 152.4 92.71 90)
+		(at 150.876 91.44 0)
 		(unit 1)
 		(exclude_from_sim no)
@@
 		(dnp no)
 		(property "Reference" "#PWR033"
-			(at 156.21 92.71 0)
+			(at 150.876 95.25 0)
 			(effects
 				(font
@@
 		)
 		(property "Value" "VBUS"
-			(at 149.1488 92.329 90)
+			(at 151.257 88.1888 90)
 			(effects
 				(font
@@
 		)
 		(property "Footprint" ""
-			(at 152.4 92.71 0)
+			(at 150.876 91.44 0)
 			(effects
 				(font
@@
 		)
 		(property "Datasheet" ""
-			(at 152.4 92.71 0)
-			(effects
-				(font
-					(size 1.27 1.27)
-				)
-				(hide yes)
-			)
-		)
-		(property "Description" ""
-			(at 152.4 92.71 0)
-			(effects
-				(font
+			(at 150.876 91.44 0)
+			(effects
+				(font
+					(size 1.27 1.27)
+				)
+				(hide yes)
+			)
+		)
+		(property "Description" ""
+			(at 150.876 91.44 0)
+			(effects
+				(font

Commit message: updated jumpers and silkscreen labelling
Changed lines of the file:
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@@
 (kicad_sch
-	(version 20231120)
+	(version 20250114)
 	(generator "eeschema")
-	(generator_version "8.0")
+	(generator_version "9.0")
 	(paper "A4")
 	(junction
@@
 	(label "Data+"
 		(at 134.62 134.62 90)
-		(fields_autoplaced yes)
 		(effects
 			(font
@@
 	(label "VBUS"
 		(at 129.54 134.62 90)
-		(fields_autoplaced yes)
 		(effects
 			(font
@@
 	(label "Data+"
 		(at 44.45 104.14 0)
-		(fields_autoplaced yes)
 		(effects
 			(font
@@
 	(label "Data-"
 		(at 44.45 99.06 0)
-		(fields_autoplaced yes)
 		(effects
 			(font
@@
 	(label "Data-"
 		(at 132.08 134.62 90)
-		(fields_autoplaced yes)
 		(effects
 			(font
@@
 	(label "Data-"
 		(at 116.84 102.87 0)
-		(fields_autoplaced yes)
 		(effects
 			(font
@@
 	(label "Data+"
 		(at 116.84 107.95 0)
-		(fields_autoplaced yes)
 		(effects
 			(font
@@
 		(shape bidirectional)
 		(at 44.45 99.06 180)
-		(fields_autoplaced yes)
 		(effects
 			(font
@@
 		(shape bidirectional)
 		(at 44.45 104.14 180)
-		(fields_autoplaced yes)
-		(effects
-			(font
+		(effects
+			(font

Commit message: tidy up schematic and bom
Parts:
- D502: renamed from USBLED1; value WHITE_LED -> LED_WHITE
- R501: renamed from R11; value 5.1k -> 5.1kΩ
- R502: renamed from R12; value 5.1k -> 5.1kΩ
- R503: renamed from R13; value 5.1k -> 5.1kΩ
- TP501: renamed from TP1; now left out of the parts list
- TP502: renamed from TP2; now left out of the parts list
- renumbered D2 to D501, J2 to J501
Changed lines of the file:
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@@
 		(on_board yes)
 		(dnp no)
-		(property "Reference" "#PWR031"
+		(property "Reference" "#PWR0503"
 			(at 128.778 103.124 0)
 			(effects
@@
 			(project "Ricardo-Kermit-Mini"
 				(path "/7db990e4-92e1-4f99-b4d2-435bbec1ba83/00000000-0000-0000-0000-000061925999"
-					(reference "#PWR031")
+					(reference "#PWR0503")
 					(unit 1)
 				)
@@
 		(on_board yes)
 		(dnp no)
-		(property "Reference" "R12"
+		(property "Reference" "R502"
 			(at 124.968 101.092 90)
 			(effects
@@
 			)
 		)
-		(property "Value" "5.1k"
+		(property "Value" "5.1kΩ"
 			(at 124.968 103.4034 90)
 			(effects
@@
 			(project "Ricardo-Kermit-Mini"
 				(path "/7db990e4-92e1-4f99-b4d2-435bbec1ba83/00000000-0000-0000-0000-000061925999"
-					(reference "R12")
+					(reference "R502")
 					(unit 1)
 				)
@@
 		(on_board yes)
 		(dnp no)
-		(property "Reference" "R11"
+		(property "Reference" "R501"
 			(at 123.19 89.0016 90)
 			(effects
@@
 			)
 		)
-		(property "Value" "5.1k"
+		(property "Value" "5.1kΩ"
 			(at 123.19 91.313 90)
 			(effects
@@
 			(project "Ricardo-Kermit-Mini"
 				(path "/7db990e4-92e1-4f99-b4d2-435bbec1ba83/00000000-0000-0000-0000-000061925999"
-					(reference "R11")
+					(reference "R501")
 					(unit 1)
 				)
@@
 		(on_board yes)
 		(dnp no)
-		(property "Reference" "#PWR029"
+		(property "Reference" "#PWR0501"
 			(at 96.52 137.16 0)
 			(effects
@@
 			(project "Ricardo-Kermit-Mini"
 				(path "/7db990e4-92e1-4f99-b4d2-435bbec1ba83/00000000-0000-0000-0000-000061925999"
-					(reference "#PWR029")
+					(reference "#PWR0501")
 					(unit 1)
 				)
@@
 		(on_board yes)
 		(dnp no)
-		(property "Reference" "J2"
+		(property "Reference" "J501"
 			(at 103.0478 82.1182 0)
 			(effects
@@
 			(project "Ricardo-Kermit-Mini"
 				(path "/7db990e4-92e1-4f99-b4d2-435bbec1ba83/00000000-0000-0000-0000-000061925999"
-					(reference "J2")
+					(reference "J501")
 					(unit 1)
 				)
@@
 		(on_board yes)
 		(dnp no)
-		(property "Reference" "#PWR032"
+		(property "Reference" "#PWR0504"
 			(at 132.08 151.13 0)
 			(effects
@@
 			(project "Ricardo-Kermit-Mini"
 				(path "/7db990e4-92e1-4f99-b4d2-435bbec1ba83/00000000-0000-0000-0000-000061925999"
-					(reference "#PWR032")
+					(reference "#PWR0504")
 					(unit 1)
 				)
@@
 		(on_board yes)
 		(dnp no)
-		(property "Reference" "D2"
+		(property "Reference" "D501"
 			(at 137.287 138.5316 0)
 			(effects
@@
 			(project "Ricardo-Kermit-Mini"
 				(path "/7db990e4-92e1-4f99-b4d2-435bbec1ba83/00000000-0000-0000-0000-000061925999"
-					(reference "D2")
+					(reference "D501")
 					(unit 1)
 				)
@@
 		(on_board yes)
 		(dnp no)
-		(property "Reference" "#PWR030"
+		(property "Reference" "#PWR0502"
 			(at 116.84 88.9 0)
 			(effects
@@
 			(project "Ricardo-Kermit-Mini"
 				(path "/7db990e4-92e1-4f99-b4d2-435bbec1ba83/00000000-0000-0000-0000-000061925999"
-					(reference "#PWR030")
+					(reference "#PWR0502")
 					(unit 1)
 				)
@@
 		(unit 1)
 		(exclude_from_sim no)
-		(in_bom yes)
-		(on_board yes)
-		(dnp no)
-		(property "Reference" "TP1"
+		(in_bom no)
+		(on_board yes)
+		(dnp no)
+		(property "Reference" "TP501"
 			(at 56.8452 97.8916 90)
 			(effects
@@
 			(project "Ricardo-Kermit-Mini"
 				(path "/7db990e4-92e1-4f99-b4d2-435bbec1ba83/00000000-0000-0000-0000-000061925999"
-					(reference "TP1")
+					(reference "TP501")
 					(unit 1)
 				)
@@
 		(unit 1)
 		(exclude_from_sim no)
-		(in_bom yes)
-		(on_board yes)
-		(dnp no)
-		(property "Reference" "TP2"
+		(in_bom no)
+		(on_board yes)
+		(dnp no)
+		(property "Reference" "TP502"
 			(at 56.8452 102.9716 90)
 			(effects
@@
 			(project "Ricardo-Kermit-Mini"
 				(path "/7db990e4-92e1-4f99-b4d2-435bbec1ba83/00000000-0000-0000-0000-000061925999"
-					(reference "TP2")
+					(reference "TP502")
 					(unit 1)
 				)
@@
 		(on_board yes)
 		(dnp no)
-		(property "Reference" "USBLED1"
+		(property "Reference" "D502"
 			(at 162.56 87.503 0)
 			(effects
@@
 			)
 		)
-		(property "Value" "WHITE_LED"
+		(property "Value" "LED_WHITE"
 			(at 162.56 89.8144 0)
 			(effects
@@
 			(project "Ricardo-Kermit-Mini"
 				(path "/7db990e4-92e1-4f99-b4d2-435bbec1ba83/00000000-0000-0000-0000-000061925999"
-					(reference "USBLED1")
+					(reference "D502")
 					(unit 1)
 				)
@@
 		(on_board yes)
 		(dnp no)
-		(property "Reference" "R13"
+		(property "Reference" "R503"
 			(at 154.94 95.3516 90)
 			(effects
@@
 			)
 		)
-		(property "Value" "5.1k"
+		(property "Value" "5.1kΩ"
 			(at 154.94 97.663 90)
 			(effects
@@
 			(project "Ricardo-Kermit-Mini"
 				(path "/7db990e4-92e1-4f99-b4d2-435bbec1ba83/00000000-0000-0000-0000-000061925999"
-					(reference "R13")
+					(reference "R503")
 					(unit 1)
 				)
@@
 		(on_board yes)
 		(dnp no)
-		(property "Reference" "#PWR034"
+		(property "Reference" "#PWR0506"
 			(at 165.1 99.06 0)
 			(effects
@@
 			(project "Ricardo-Kermit-Mini"
 				(path "/7db990e4-92e1-4f99-b4d2-435bbec1ba83/00000000-0000-0000-0000-000061925999"
-					(reference "#PWR034")
+					(reference "#PWR0506")
 					(unit 1)
 				)
@@
 		(on_board yes)
 		(dnp no)
-		(property "Reference" "#PWR033"
+		(property "Reference" "#PWR0505"
 			(at 150.876 95.25 0)
 			(effects
@@
 			(project "Ricardo-Kermit-Mini"
 				(path "/7db990e4-92e1-4f99-b4d2-435bbec1ba83/00000000-0000-0000-0000-000061925999"
-					(reference "#PWR033")
-					(unit 1)
-				)
+					(reference "#PWR0505")
+					(unit 1)
+				)

Commit message: continued
Parts:
- D502: footprint Resistor_SMD:R_0402_1005Metric -> LED_SMD:LED_0402_1005Metric
Changed lines of the file:
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@@
 			)
 		)
-		(property "Footprint" "Resistor_SMD:R_0402_1005Metric"
+		(property "Footprint" "LED_SMD:LED_0402_1005Metric"
 			(at 162.56 92.71 90)
 			(effects
